File: Paul/project/Paul.kicad_pcb (KiCad board)
At the start: 2 copper layers, 76.2 x 25.4 mm, 43 parts, among them J1 USB_C_Receptacle_USB2.0_16P

Commit message: remove logo
Parts:
- removed G***: LOGO, custom:controls_logo_50x16mm
- removed G***: LOGO, custom:bnl_logo_new_12.4x3.0mm
