File: SidSky/project/SidSky.kicad_pcb (KiCad board)
At the start: 2 copper layers, 76.2 x 25.4 mm, 41 parts, among them J1 USB_C_Receptacle_USB2.0_16P

Commit message: routing
Parts:
- added GND1: GND, TestPoint:TestPoint_Pad_D1.0mm, F.Cu at (160.8, 78.1)
- moved +5V_fuse1 3.64 mm to (154.0, 74.5)
Routing:
- net Net-(D9-A): track 0.23 -> 23.8 mm, vias 0 -> 1
- net Net-(D7-A): track 0.00 -> 15.6 mm, vias 0 -> 1
- net Net-(D17-A): track 0.00 -> 14.4 mm, vias 0 -> 1
- net Net-(D16-A): track 0.00 -> 14.1 mm, vias 0 -> 1
- net Net-(D2-A): track 0.00 -> 13.2 mm, vias 0 -> 1
- net GND: track 194.7 -> 206.2 mm, vias 0 -> 1
- net Net-(D3-A): track 0.00 -> 10.6 mm, vias 0 -> 1
- net Net-(D15-A): track 0.00 -> 10.4 mm, vias 0 -> 1
- net Net-(D10-A): track 0.00 -> 7.52 mm, vias 0 -> 1
- net Net-(D14-A): track 0.00 -> 7.46 mm, vias 0 -> 1
- net Net-(D6-A): track 0.00 -> 6.79 mm, vias 0 -> 1
- net Net-(D8-A): track 0.00 -> 6.57 mm, vias 0 -> 1
- net Net-(D12-A): track 0.00 -> 5.54 mm, vias 0 -> 1
- net Net-(D5-A): track 0.00 -> 5.50 mm, vias 0 -> 1
- net Net-(D11-A): track 0.00 -> 5.05 mm, vias 0 -> 1
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Other:
- board text added: "Bless this home and all who enter"
- board text removed: "Bless this home and all those who enter"
